File: 3886_3/3886_3.kicad_pcb (KiCad board)
At the start: 2 copper layers, 95 x 78 mm, 59 parts, among them J101 2, J102 2, J103 3, Q101 BT139-600E, Q102 BC817, Q103 BC807, U101 LM3886TF

Commit message: Add files via upload
Parts:
- R119, R120: value 10 -> 1
Routing:
- net GND: track 240.8 -> 229.8 mm
Changed lines of the file:
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@@
 			)
 		)
-		(property "Value" "10"
+		(property "Value" "1"
 			(at 0 -1.83 0)
 			(layer "B.Fab")
@@
 			)
 		)
-		(property "Value" "10"
+		(property "Value" "1"
 			(at 0 -1.83 0)
 			(layer "B.Fab")
@@
 	)
 	(gr_line
-		(start 109.728 60.706)
+		(start 100.33 60.706)
 		(end 94.5515 60.706)
 		(stroke
@@
 	)
 	(segment
-		(start 111.633 60.96)
+		(start 102.362 60.96)
 		(end 92.583 60.96)
 		(width 0.75)
@@
 	)
 	(via
-		(at 111.633 60.96)
+		(at 102.362 60.96)
 		(size 2.5)
 		(drill 0.8)
@@
 	)
 	(segment
-		(start 112.903 60.96)
-		(end 111.633 60.96)
-		(width 0.75)
-		(layer "B.Cu")
-		(net 2)
-	)
-	(segment
 		(start 80.01 49.784)
 		(end 78.323 49.784)
@@
 		(layer "B.Cu")
 		(net 2)
-	)
-	(segment
-		(start 113.284 61.341)
-		(end 112.903 60.96)
-		(width 0.75)
-		(layer "B.Cu")
-		(net 2)
