File: 3886_3/3886_3.kicad_pcb (KiCad board)
At the start: 2 copper layers, 95 x 78 mm, 57 parts, among them J101 2, J102 2, J103 3, Q101 BT139-600E, Q102 BC817, Q103 BC807, U101 LM3886TF

Commit message: Add files via upload
Parts:
- moved C105 1.41 mm to (89.9, 46.7)
Routing:
- net Net-(U101--): track 21.6 -> 23.3 mm
Changed lines of the file:
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@@
 	(footprint "Capacitor_THT:C_Rect_L7.0mm_W2.5mm_P5.00mm"
 		(layer "F.Cu")
-		(at 88.519 46.903 -90)
+		(at 89.916 46.736 -90)
 		(descr "C, Rect series, Radial, pin pitch=5.00mm, length*width=7*2.5mm^2, Capacitor")
 		(tags "C Rect series Radial pin pitch 5.00mm length 7mm width 2.5mm Capacitor")
@@
 	)
 	(segment
+		(start 108.458 97.282)
+		(end 88.0618 97.282)
+		(width 1.5)
+		(layer "B.Cu")
+		(net 2)
+	)
+	(segment
 		(start 80.238 68.453)
 		(end 80.238 66.583)
@@
 	)
 	(segment
-		(start 112.776 92.964)
-		(end 108.712 97.028)
-		(width 1.5)
+		(start 80.238 66.583)
+		(end 80.212 66.557)
+		(width 0.5)
 		(layer "B.Cu")
 		(net 2)
 	)
 	(segment
-		(start 93.218 55.499)
-		(end 101.6 55.499)
-		(width 0.75)
+		(start 112.776 92.964)
+		(end 108.458 97.282)
+		(width 1.5)
 		(layer "B.Cu")
 		(net 2)
 	)
 	(segment
-		(start 80.238 66.583)
-		(end 80.212 66.557)
-		(width 0.5)
+		(start 83.2358 48.9712)
+		(end 90.7542 48.9712)
+		(width 0.75)
 		(layer "B.Cu")
 		(net 2)
 	)
 	(segment
-		(start 83.2358 48.9712)
-		(end 90.1192 48.9712)
-		(width 0.75)
+		(start 88.0618 97.282)
+		(end 81.9658 91.186)
+		(width 1.5)
 		(layer "B.Cu")
 		(net 2)
@@
 		(start 119.888 78.232)
 		(end 120.904 79.248)
-		(width 2)
+		(width 1.5)
 		(layer "B.Cu")
 		(net 2)
@@
 	)
 	(segment
+		(start 116.84 78.232)
+		(end 113.792 78.232)
+		(width 1.5)
+		(layer "B.Cu")
+		(net 2)
+	)
+	(segment
 		(start 97.536 44.45)
 		(end 97.536 47.244)
@@
 	)
 	(segment
+		(start 113.792 78.232)
+		(end 112.776 79.248)
+		(width 1.5)
+		(layer "B.Cu")
+		(net 2)
+	)
+	(segment
 		(start 84.074 44.069)
 		(end 82.7786 44.069)
@@
 	)
 	(segment
-		(start 116.84 78.232)
-		(end 113.792 78.232)
-		(width 2)
-		(layer "B.Cu")
-		(net 2)
-	)
-	(segment
 		(start 86.36 65.278)
 		(end 85.081 66.557)
@@
 		(start 116.84 78.232)
 		(end 119.888 78.232)
-		(width 2)
+		(width 1.5)
 		(layer "B.Cu")
 		(net 2)
@@
 	)
 	(segment
+		(start 92.202 50.419)
+		(end 92.202 53.848)
+		(width 0.75)
+		(layer "B.Cu")
+		(net 2)
+	)
+	(segment
 		(start 78.323 51.108)
 		(end 78.323 49.784)
@@
 	)
 	(segment
-		(start 87.8078 97.028)
-		(end 81.9658 91.186)
-		(width 1.5)
-		(layer "B.Cu")
-		(net 2)
-	)
-	(segment
 		(start 66.1924 47.5996)
 		(end 66.167 47.625)
@@
 	)
 	(segment
-		(start 120.904 79.248)
-		(end 120.904 92.71)
-		(width 2)
+		(start 112.776 79.248)
+		(end 112.776 92.964)
+		(width 1.5)
 		(layer "B.Cu")
 		(net 2)
 	)
 	(segment
-		(start 108.712 97.028)
-		(end 87.8078 97.028)
-		(width 1.5)
+		(start 92.202 53.848)
+		(end 93.853 55.499)
+		(width 0.75)
 		(layer "B.Cu")
 		(net 2)
 	)
 	(segment
-		(start 83.312 70.349)
-		(end 83.33 70.367)
+		(start 90.7542 48.9712)
+		(end 92.202 50.419)
 		(width 0.75)
 		(layer "B.Cu")
@@
 	)
 	(segment
-		(start 81.7372 45.1104)
-		(end 81.7372 46.9138)
-		(width 0.35)
+		(start 120.904 79.248)
+		(end 120.904 92.71)
+		(width 1.5)
 		(layer "B.Cu")
 		(net 2)
 	)
 	(segment
-		(start 90.1192 48.9712)
-		(end 91.567 50.419)
+		(start 83.312 70.349)
+		(end 83.33 70.367)
 		(width 0.75)
 		(layer "B.Cu")
@@
 	)
 	(segment
-		(start 88.392 60.96)
-		(end 86.36 62.992)
-		(width 1)
+		(start 81.7372 45.1104)
+		(end 81.7372 46.9138)
+		(width 0.35)
 		(layer "B.Cu")
 		(net 2)
 	)
 	(segment
-		(start 91.567 53.848)
-		(end 93.218 55.499)
-		(width 0.75)
+		(start 88.392 60.96)
+		(end 86.36 62.992)
+		(width 1)
 		(layer "B.Cu")
 		(net 2)
@@
 	)
 	(segment
-		(start 112.776 79.248)
-		(end 112.776 92.964)
-		(width 2)
-		(layer "B.Cu")
-		(net 2)
-	)
-	(segment
 		(start 83.1342 48.9712)
 		(end 80.7466 48.9712)
@@
 	)
 	(segment
-		(start 81.7372 46.9138)
-		(end 81.0514 47.5996)
-		(width 0.35)
-		(layer "B.Cu")
-		(net 2)
-	)
-	(segment
-		(start 113.792 78.232)
-		(end 112.776 79.248)
-		(width 2)
+		(start 93.853 55.499)
+		(end 101.6 55.499)
+		(width 0.75)
 		(layer "B.Cu")
 		(net 2)
 	)
 	(segment
-		(start 91.567 50.419)
-		(end 91.567 53.848)
-		(width 0.75)
+		(start 81.7372 46.9138)
+		(end 81.0514 47.5996)
+		(width 0.35)
 		(layer "B.Cu")
 		(net 2)
@@
 	)
 	(segment
-		(start 84.836 55.626)
-		(end 84.328 55.626)
-		(width 2)
-		(layer "B.Cu")
-		(net 8)
-	)
-	(segment
-		(start 88.392 52.07)
-		(end 84.836 55.626)
-		(width 2)
-		(layer "B.Cu")
-		(net 8)
-	)
-	(segment
 		(start 84.328 61.214)
 		(end 84.582 61.468)
@@
 	)
 	(segment
+		(start 88.726 51.736)
+		(end 84.836 55.626)
+		(width 2)
+		(layer "B.Cu")
+		(net 8)
+	)
+	(segment
 		(start 81.723 53.021)
 		(end 84.328 55.626)
@@
 	)
 	(segment
+		(start 89.916 51.736)
+		(end 88.726 51.736)
+		(width 2)
+		(layer "B.Cu")
+		(net 8)
+	)
+	(segment
 		(start 87.122 58.166)
 		(end 85.09 58.166)
@@
 	)
 	(segment
+		(start 84.836 55.626)
+		(end 84.328 55.626)
+		(width 2)
+		(layer "B.Cu")
+		(net 8)
+	)
+	(segment
 		(start 84.328 55.626)
 		(end 84.328 58.674)
@@
 		(start 116.84 94.488)
 		(end 116.84 80.732)
-		(width 2)
+		(width 1.5)
 		(layer "B.Cu")
 		(net 12)
@@
 		(start 86.36 99.822)
 		(end 94.234 99.822)
-		(width 1.5)
+		(width 2)
 		(layer "B.Cu")
 		(net 24)
@@
 				(xy 100.838 62.992) (xy 100.838 50.038) (xy 103.124 50.038) (xy 103.124 41.783) (xy 66.421 41.783)
 				(xy 66.421 55.372) (xy 59.182 55.372) (xy 59.182 59.944) (xy 52.578 59.944) (xy 52.578 65.532) (xy 57.15 65.532)
-				(xy 58.674 67.056) (xy 58.674 68.58) (xy 63.5 73.406) (xy 65.278 73.406) (xy 79.756 73.406) (xy 82.55 75.946)
-				(xy 82.55 90.678) (xy 82.55 120.65) (xy 124.46 120.65) (xy 124.46 62.738)
+				(xy 58.674 67.056) (xy 58.674 68.58) (xy 64.008 73.914) (xy 79.248 73.914) (xy 82.55 77.47) (xy 82.55 90.678)
+				(xy 82.55 120.65) (xy 124.46 120.65) (xy 124.46 62.738)
 			)
 		)
@@
 		(min_thickness 0.25)
 		(filled_areas_thickness no)
-		(fill
+		(fill yes
 			(thermal_gap 0.5)
 			(thermal_bridge_width 0.5)

Commit message: Add files via upload
Parts:
- removed R101: 0, Resistor_SMD:R_1206_3216Metric_Pad1.30x1.75mm_HandSolder
- moved C107 0.51 mm to (97.5, 46.7)
- moved C102 0.38 mm to (99.8, 52.8)
Connections:
- J101 pad 1: Net-(J101-Pin_1) -> GND
Routing:
- net Net-(J101-Pin_1): track 9.12 -> 0.00 mm
- net GND: track 229.9 -> 226.5 mm
- net Net-(U101-MUTE): track 28.2 -> 27.6 mm

Commit message: Add files via upload
Parts:
- moved R102 2.54 mm to (108.7, 45.5)
- moved C107 0.81 mm to (98.3, 46.8)
- moved R111 0.25 mm to (85.6, 117.9)
Routing:
- net Net-(C101-Pad2): track 16.9 -> 13.9 mm
- net GND: track 226.5 -> 228.3 mm
- net Net-(U101-MUTE): track 27.6 -> 28.4 mm
- net VP: track 79.5 -> 78.8 mm
- net Net-(U101-+): track 19.7 -> 20.5 mm

Commit message: Add files via upload
Parts:
- moved R113 1.14 mm to (99.2, 99.8)
- moved R112 0.76 mm to (99.2, 103.8)
- moved R114 0.65 mm to (106.0, 101.7)
Routing:
- net Net-(D101-A): track 20.1 -> 21.5 mm
Changed lines of the file:
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@@
 		(tags "C Rect series Radial pin pitch 27.50mm length 31.5mm width 13mm Capacitor")
 		(property "Reference" "C104"
-			(at -3.556 5.588 180)
+			(at -3.556 4.826 180)
 			(layer "F.SilkS")
 			(effects
@@
 		(tags "C Rect series Radial pin pitch 27.50mm length 31.5mm width 13mm Capacitor")
 		(property "Reference" "C103"
-			(at -3.556 5.842 180)
+			(at -3.556 5.08 180)
 			(layer "F.SilkS")
 			(effects
@@
 		(tags "TO-220-3 Vertical RM 2.54mm")
 		(property "Reference" "Q101"
-			(at 2.413 4.445 180)
+			(at 2.413 4.826 180)
 			(layer "F.SilkS")
 			(effects
@@
 	(footprint "Resistor_SMD:R_1206_3216Metric_Pad1.30x1.75mm_HandSolder"
 		(layer "B.Cu")
-		(at 105.918 102.362)
+		(at 106.045 101.727)
 		(descr "Resistor SMD 1206 (3216 Metric), square (rectangular) end terminal, IPC-7351 nominal with elongated pad for handsoldering. (Body size source: IPC-SM-782 page 72, https://www.pcb-3d.com/wordpress/wp-content/uploads/ipc-sm-782a_amendment_1_and_2.pdf), generated with kicad-footprint-generator")
 		(tags "resistor handsolder")
@@
 	(footprint "Resistor_SMD:R_1206_3216Metric_Pad1.30x1.75mm_HandSolder"
 		(layer "B.Cu")
-		(at 99.187 100.965)
+		(at 99.187 99.822)
 		(descr "Resistor SMD 1206 (3216 Metric), square (rectangular) end terminal, IPC-7351 nominal with elongated pad for handsoldering. (Body size source: IPC-SM-782 page 72, https://www.pcb-3d.com/wordpress/wp-content/uploads/ipc-sm-782a_amendment_1_and_2.pdf), generated with kicad-footprint-generator")
 		(tags "resistor handsolder")
@@
 	(footprint "Resistor_SMD:R_1206_3216Metric_Pad1.30x1.75mm_HandSolder"
 		(layer "B.Cu")
-		(at 99.187 104.521)
+		(at 99.187 103.759)
 		(descr "Resistor SMD 1206 (3216 Metric), square (rectangular) end terminal, IPC-7351 nominal with elongated pad for handsoldering. (Body size source: IPC-SM-782 page 72, https://www.pcb-3d.com/wordpress/wp-content/uploads/ipc-sm-782a_amendment_1_and_2.pdf), generated with kicad-footprint-generator")
 		(tags "resistor handsolder")
@@
 	)
 	(gr_line
-		(start 59.182 60.325)
-		(end 59.182 52.451)
+		(start 59.309 60.325)
+		(end 59.309 52.451)
 		(stroke
 			(width 0.8)
@@
 	)
 	(gr_line
-		(start 35.941 63.246)
-		(end 41.91 63.246)
+		(start 35.941 63.119)
+		(end 41.91 63.119)
 		(stroke
 			(width 0.8)
@@
 	)
 	(gr_line
-		(start 100.33 60.706)
-		(end 93.853 60.706)
+		(start 100.33 60.579)
+		(end 93.853 60.579)
 		(stroke
 			(width 0.8)
@@
 	)
 	(segment
-		(start 112.776 79.248)
-		(end 112.776 93.726)
-		(width 1.5)
-		(layer "B.Cu")
-		(net 2)
-	)
-	(segment
 		(start 58.928 62.992)
 		(end 64.389 68.453)
@@
 	)
 	(segment
-		(start 81.7372 46.9138)
-		(end 81.0514 47.5996)
-		(width 0.35)
+		(start 113.792 78.232)
+		(end 112.776 79.248)
+		(width 1.5)
 		(layer "B.Cu")
 		(net 2)
 	)
 	(segment
-		(start 112.776 93.726)
-		(end 109.22 97.282)
-		(width 1.5)
+		(start 81.7372 46.9138)
+		(end 81.0514 47.5996)
+		(width 0.35)
 		(layer "B.Cu")
 		(net 2)
@@
 	)
 	(segment
-		(start 109.22 97.282)
-		(end 88.0618 97.282)
-		(width 1.5)
+		(start 93.218 55.372)
+		(end 101.6 55.372)
+		(width 0.75)
 		(layer "B.Cu")
 		(net 2)
 	)
 	(segment
-		(start 93.218 55.372)
-		(end 101.6 55.372)
-		(width 0.75)
+		(start 109.728 96.774)
+		(end 87.5538 96.774)
+		(width 1.5)
 		(layer "B.Cu")
 		(net 2)
@@
 	)
 	(segment
-		(start 88.0618 97.282)
-		(end 81.9658 91.186)
-		(width 1.5)
-		(layer "B.Cu")
-		(net 2)
-	)
-	(segment
 		(start 86.36 65.278)
 		(end 85.081 66.557)
@@
 	)
 	(segment
+		(start 112.776 93.726)
+		(end 109.728 96.774)
+		(width 1.5)
+		(layer "B.Cu")
+		(net 2)
+	)
+	(segment
 		(start 80.7466 48.9712)
 		(end 79.9338 49.784)
@@
 	)
 	(segment
-		(start 113.792 78.232)
-		(end 112.776 79.248)
+		(start 87.5538 96.774)
+		(end 81.9658 91.186)
 		(width 1.5)
 		(layer "B.Cu")
@@
 	)
 	(segment
+		(start 112.776 79.248)
+		(end 112.776 93.726)
+		(width 1.5)
+		(layer "B.Cu")
+		(net 2)
+	)
+	(segment
 		(start 117.856 66.548)
 		(end 118.618 67.31)
@@
 	)
 	(segment
-		(start 108.712 102.362)
-		(end 110.871 100.203)
+		(start 110.617 100.203)
+		(end 114.808 100.203)
 		(width 0.75)
 		(layer "B.Cu")
@@
 	)
 	(segment
-		(start 107.468 102.362)
-		(end 108.712 102.362)
+		(start 118.136 98.324)
+		(end 116.84 97.028)
 		(width 0.75)
 		(layer "B.Cu")
@@
 	)
 	(segment
-		(start 118.136 98.324)
-		(end 116.84 97.028)
+		(start 109.093 101.727)
+		(end 110.617 100.203)
 		(width 0.75)
 		(layer "B.Cu")
@@
 	)
 	(segment
+		(start 107.595 101.727)
+		(end 109.093 101.727)
+		(width 0.75)
+		(layer "B.Cu")
+		(net 13)
+	)
+	(segment
 		(start 114.808 100.203)
 		(end 118.364 100.203)
@@
 	)
 	(segment
-		(start 110.871 100.203)
-		(end 114.808 100.203)
+		(start 100.737 104.521)
+		(end 100.711 104.547)
 		(width 0.75)
 		(layer "B.Cu")
-		(net 13)
+		(net 14)
 	)
 	(segment
 		(start 102.616 102.362)
-		(end 102.616 104.013)
+		(end 102.616 103.378)
 		(width 0.75)
 		(layer "B.Cu")
@@
 	)
 	(segment
-		(start 102.108 100.965)
-		(end 102.616 101.473)
+		(start 102.235 103.759)
+		(end 100.737 103.759)
 		(width 0.75)
 		(layer "B.Cu")
@@
 	)
 	(segment
-		(start 100.711 104.547)
-		(end 100.711 108.204)
+		(start 100.737 103.759)
+		(end 100.737 104.521)
 		(width 0.75)
 		(layer "B.Cu")
@@
 	)
 	(segment
-		(start 98.378 108.204)
-		(end 98.806 108.632)
-		(width 2.5)
+		(start 100.737 99.822)
+		(end 102.235 99.822)
+		(width 0.75)
 		(layer "B.Cu")
 		(net 14)
 	)
 	(segment
-		(start 104.368 102.362)
-		(end 102.616 102.362)
+		(start 104.495 101.727)
+		(end 102.616 101.727)
 		(width 0.75)
 		(layer "B.Cu")
@@
 	)
 	(segment
-		(start 102.108 104.521)
-		(end 100.737 104.521)
-		(width 0.75)
+		(start 98.378 108.204)
+		(end 98.806 108.632)
+		(width 2.5)
 		(layer "B.Cu")
 		(net 14)
 	)
 	(segment
-		(start 100.737 100.965)
-		(end 102.108 100.965)
+		(start 102.235 99.822)
+		(end 102.616 100.203)
 		(width 0.75)
 		(layer "B.Cu")
@@
 	)
 	(segment
-		(start 98.806 108.632)
-		(end 98.806 112.95)
-		(width 1.5)
+		(start 102.616 103.378)
+		(end 102.235 103.759)
+		(width 0.75)
 		(layer "B.Cu")
 		(net 14)
 	)
 	(segment
-		(start 102.616 104.013)
-		(end 102.108 104.521)
-		(width 0.75)
+		(start 98.806 108.632)
+		(end 98.806 112.95)
+		(width 1.5)
 		(layer "B.Cu")
 		(net 14)
 	)
 	(segment
-		(start 102.616 101.473)
-		(end 102.616 102.362)
+		(start 100.711 104.547)
+		(end 100.711 108.204)
 		(width 0.75)
 		(layer "B.Cu")
@@
 	)
 	(segment
-		(start 100.737 104.521)
-		(end 100.711 104.547)
+		(start 102.616 100.203)
+		(end 102.616 102.362)
 		(width 0.75)
 		(layer "B.Cu")
@@
 	)
 	(segment
-		(start 94.234 99.822)
-		(end 95.377 100.965)
-		(width 1)
-		(layer "B.Cu")
-		(net 23)
-	)
-	(segment
-		(start 97.663 100.991)
-		(end 97.663 103.987)
-		(width 0.75)
-		(layer "B.Cu")
-		(net 23)
-	)
-	(segment
-		(start 97.637 101.372)
-		(end 97.637 100.965)
+		(start 97.663 99.848)
+		(end 97.663 103.733)
 		(width 0.75)
 		(layer "B.Cu")
@@
 	)
 	(segment
-		(start 97.637 100.965)
-		(end 97.663 100.991)
-		(width 0.75)
+		(start 86.36 99.822)
+		(end 94.234 99.822)
+		(width 3.5)
 		(layer "B.Cu")
 		(net 23)
 	)
 	(segment
-		(start 95.377 100.965)
-		(end 97.637 100.965)
-		(width 1)
+		(start 73.152 91.186)
+		(end 77.724 91.186)
+		(width 3)
 		(layer "B.Cu")
 		(net 23)
 	)
 	(segment
-		(start 86.36 99.822)
-		(end 94.234 99.822)
-		(width 2)
+		(start 94.234 99.822)
+		(end 97.637 99.822)
+		(width 1)
 		(layer "B.Cu")
 		(net 23)
 	)
 	(segment
-		(start 73.152 91.186)
-		(end 77.724 91.186)
-		(width 3)
+		(start 97.637 99.822)
+		(end 97.663 99.848)
+		(width 0.75)
 		(layer "B.Cu")
 		(net 23)
 	)
 	(segment
-		(start 97.663 103.987)
-		(end 97.637 104.013)
+		(start 97.663 103.733)
+		(end 97.637 103.759)
 		(width 0.75)
 		(layer "B.Cu")
@@
 		(layer "B.Cu")
 		(net 23)
-	)
-	(segment
-		(start 97.637 104.013)
-		(end 97.637 104.521)
-		(width 0.75)
-		(layer "B.Cu")
-		(net 23)

Commit message: Add files via upload
Parts:
- moved C106 1.27 mm to (80.4, 61.2)
Routing:
- net VP: track 78.8 -> 83.1 mm
- net Net-(C106-Pad1): track 6.16 -> 4.89 mm
- net Net-(U101--): track 23.3 -> 24.2 mm
- net GND: track 227.8 -> 228.6 mm
Changed lines of the file:
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@@
 		(tags "Resistor Axial_DIN0207 series Axial Horizontal pin pitch 10.16mm 0.25W = 1/4W length 6.3mm diameter 2.5mm")
 		(property "Reference" "R104"
-			(at 3.302 2.286 0)
+			(at 5.334 2.413 0)
 			(layer "F.SilkS")
 			(effects
@@
 			(pinfunction "Pin_3")
 			(pintype "passive")
-			(thermal_bridge_width 2)
+			(thermal_bridge_width 1.5)
 		)
 		(embedded_fonts no)
@@
 			(pinfunction "Pin_1")
 			(pintype "passive")
-			(thermal_bridge_width 2)
+			(thermal_bridge_width 1.5)
 		)
 		(pad "2" thru_hole roundrect
@@
 	(footprint "Capacitor_SMD:C_1206_3216Metric_Pad1.33x1.80mm_HandSolder"
 		(layer "B.Cu")
-		(at 81.661 61.214)
+		(at 80.391 61.214)
 		(descr "Capacitor SMD 1206 (3216 Metric), square (rectangular) end terminal, IPC-7351 nominal with elongated pad for handsoldering. (Body size source: IPC-SM-782 page 76, https://www.pcb-3d.com/wordpress/wp-content/uploads/ipc-sm-782a_amendment_1_and_2.pdf), generated with kicad-footprint-generator")
 		(tags "capacitor handsolder")
 		(property "Reference" "C106"
-			(at -0.381 -1.778 180)
+			(at 0 -1.778 180)
 			(layer "B.SilkS")
 			(effects
@@
 	)
 	(gr_line
-		(start 100.33 60.579)
+		(start 101.092 60.579)
 		(end 93.853 60.579)
 		(stroke
@@
 	)
 	(segment
-		(start 102.362 60.96)
+		(start 103.124 60.96)
 		(end 91.948 60.96)
 		(width 0.75)
@@
 	)
 	(via
-		(at 102.362 60.96)
+		(at 103.124 60.96)
 		(size 2.5)
 		(drill 0.8)
@@
 	)
 	(segment
-		(start 45.7835 70.1675)
-		(end 52.07 63.881)
-		(width 3.5)
-		(layer "B.Cu")
-		(net 6)
-	)
-	(segment
 		(start 68.123 49.86)
 		(end 68.834 49.149)
@@
 	)
 	(segment
-		(start 45.7835 70.1675)
-		(end 45.72 70.231)
+		(start 52.959 61.595)
+		(end 57.658 56.896)
 		(width 4)
 		(layer "B.Cu")
@@
 	)
 	(segment
-		(start 48.4505 81.3435)
-		(end 48.4505 81.7245)
-		(width 2)
-		(layer "B.Cu")
-		(net 6)
-	)
-	(segment
-		(start 52.959 61.595)
-		(end 57.658 56.896)
-		(width 4)
+		(start 46.99 80.264)
+		(end 49.022 82.296)
+		(width 4.5)
 		(layer "B.Cu")
 		(net 6)
@@
 	)
 	(segment
-		(start 43.942 77.216)
-		(end 48.4505 81.7245)
-		(width 4)
+		(start 52.07 63.881)
+		(end 52.07 61.595)
+		(width 3.5)
 		(layer "B.Cu")
 		(net 6)
@@
 	)
 	(segment
-		(start 51.054 78.74)
-		(end 48.4505 81.3435)
-		(width 2)
-		(layer "B.Cu")
-		(net 6)
-	)
-	(segment
 		(start 56.769 56.896)
 		(end 58.547 56.896)
@@
 	)
 	(segment
-		(start 52.07 63.881)
-		(end 52.07 61.595)
-		(width 3.5)
-		(layer "B.Cu")
-		(net 6)
-	)
-	(segment
 		(start 74.041 49.022)
 		(end 74.168 49.149)
@@
 	)
 	(segment
-		(start 45.72 70.231)
-		(end 45.72 78.994)
+		(start 46.99 76.962)
+		(end 46.99 80.264)
 		(width 4)
 		(layer "B.Cu")
@@
 	)
 	(segment
+		(start 38.1 77.216)
+		(end 46.736 77.216)
+		(width 3.5)
+		(layer "B.Cu")
+		(net 6)
+	)
+	(segment
+		(start 51.054 78.74)
+		(end 49.53 80.264)
+		(width 2)
+		(layer "B.Cu")
+		(net 6)
+	)
+	(segment
 		(start 74.923 52.8898)
 		(end 74.923 49.918)
@@
 	)
 	(segment
+		(start 46.99 68.961)
+		(end 46.99 80.264)
+		(width 4)
+		(layer "B.Cu")
+		(net 6)
+	)
+	(segment
 		(start 74.168 49.149)
 		(end 74.4474 49.4284)
@@
 	)
 	(segment
+		(start 49.53 80.264)
+		(end 46.99 80.264)
+		(width 2)
+		(layer "B.Cu")
+		(net 6)
+	)
+	(segment
 		(start 68.961 49.022)
 		(end 69.215 48.768)
@@
 	)
 	(segment
-		(start 38.1 77.216)
-		(end 43.942 77.216)
+		(start 46.99 68.961)
+		(end 52.07 63.881)
+		(width 3.5)
+		(layer "B.Cu")
+		(net 6)
+	)
+	(segment
+		(start 46.736 77.216)
+		(end 46.99 76.962)
 		(width 3.5)
 		(layer "B.Cu")
@@
 	)
 	(segment
-		(start 84.328 61.214)
-		(end 84.582 61.468)
-		(width 1.5)
+		(start 81.9535 61.214)
+		(end 83.947 61.214)
+		(width 1)
 		(layer "B.Cu")
 		(net 8)
 	)
 	(segment
-		(start 84.582 61.468)
-		(end 84.582 58.928)
-		(width 1.5)
+		(start 84.582 55.88)
+		(end 84.328 55.626)
+		(width 2.5)
 		(layer "B.Cu")
 		(net 8)
@@
 	)
 	(segment
+		(start 84.582 60.579)
+		(end 84.582 58.928)
+		(width 1)
+		(layer "B.Cu")
+		(net 8)
+	)
+	(segment
 		(start 81.723 53.021)
 		(end 84.328 55.626)
@@
 	)
 	(segment
-		(start 84.328 58.674)
-		(end 84.582 58.928)
-		(width 2)
+		(start 85.09 58.166)
+		(end 84.582 58.674)
+		(width 2.5)
 		(layer "B.Cu")
 		(net 8)
 	)
 	(segment
-		(start 85.09 58.166)
-		(end 84.582 58.674)
-		(width 2.5)
+		(start 84.328 58.674)
+		(end 84.582 58.928)
+		(width 2)
 		(layer "B.Cu")
 		(net 8)
 	)
 	(segment
-		(start 83.2235 61.214)
-		(end 84.328 61.214)
-		(width 1.5)
+		(start 84.582 58.928)
+		(end 84.582 55.88)
+		(width 2.5)
 		(layer "B.Cu")
 		(net 8)
@@
 	)
 	(segment
-		(start 84.328 55.626)
-		(end 84.328 58.674)
-		(width 2.5)
+		(start 83.947 61.214)
+		(end 84.582 60.579)
+		(width 1)
 		(layer "B.Cu")
 		(net 8)
 	)
 	(segment
-		(start 78.74 56.414)
-		(end 78.74 61.468)
+		(start 78.74 61.214)
+		(end 78.8285 61.214)
 		(width 1)
 		(layer "B.Cu")
@@
 	)
 	(segment
-		(start 78.994 61.214)
-		(end 80.0985 61.214)
-		(width 1.5)
+		(start 78.74 56.414)
+		(end 78.74 61.214)
+		(width 1)
 		(layer "B.Cu")
 		(net 9)
@@
 			(pts
 				(xy 40.132 110.236) (xy 36.83 110.236) (xy 36.83 105.2576) (xy 46.1264 105.2576) (xy 50.8 100.584)
-				(xy 50.8 80.01) (xy 51.816 80.01) (xy 51.816 95.504) (xy 63.246 95.504) (xy 66.294 99.06) (xy 77.724 99.06)
+				(xy 50.8 72.644) (xy 51.816 72.644) (xy 51.816 95.504) (xy 63.246 95.504) (xy 66.294 99.06) (xy 77.724 99.06)
 				(xy 77.724 93.853) (xy 82.55 93.853) (xy 82.55 101.6) (xy 77.216 101.6) (xy 77.216 114.554) (xy 65.278 114.554)
 				(xy 65.278 116.332) (xy 46.228 116.332)
