File: 3886_3/3886_3.kicad_pcb (KiCad board)
At the start: 2 copper layers, 95 x 78 mm, 56 parts, among them J101 2, J102 2, J103 3, Q101 BT139-600E, Q102 BC817, Q103 BC807, U101 LM3886TF

Commit message: Add files via upload
Parts:
- moved R102 2.05 mm to (109.0, 47.5)
- moved R103 0.51 mm to (95.5, 52.8)
- moved C107 0.47 mm to (98.8, 46.8)
Routing:
- net Net-(C101-Pad2): track 13.9 -> 15.5 mm
Changed lines of the file:
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@@
 	(footprint "Resistor_THT:R_Axial_DIN0207_L6.3mm_D2.5mm_P10.16mm_Horizontal"
 		(layer "F.Cu")
-		(at 94.996 52.832)
+		(at 95.504 52.832)
 		(descr "Resistor, Axial_DIN0207 series, Axial, Horizontal, pin pitch=10.16mm, 0.25W = 1/4W, length*diameter=6.3*2.5mm^2, http://cdn-reichelt.de/documents/datenblatt/B400/1_4W%23YAG.pdf")
 		(tags "Resistor Axial_DIN0207 series Axial Horizontal pin pitch 10.16mm 0.25W = 1/4W length 6.3mm diameter 2.5mm")
@@
 	(footprint "Resistor_THT:R_Axial_DIN0207_L6.3mm_D2.5mm_P10.16mm_Horizontal"
 		(layer "F.Cu")
-		(at 108.712 45.466 -90)
+		(at 108.966 47.498 -90)
 		(descr "Resistor, Axial_DIN0207 series, Axial, Horizontal, pin pitch=10.16mm, 0.25W = 1/4W, length*diameter=6.3*2.5mm^2, http://cdn-reichelt.de/documents/datenblatt/B400/1_4W%23YAG.pdf")
 		(tags "Resistor Axial_DIN0207 series Axial Horizontal pin pitch 10.16mm 0.25W = 1/4W length 6.3mm diameter 2.5mm")
 		(property "Reference" "R102"
-			(at 3.429 2.413 90)
+			(at 1.778 2.413 90)
 			(layer "F.SilkS")
 			(effects
@@
 	(footprint "Capacitor_THT:CP_Radial_D6.3mm_P2.50mm"
 		(layer "F.Cu")
-		(at 98.338 46.843)
+		(at 98.806 46.843)
 		(descr "CP, Radial series, Radial, pin pitch=2.50mm, diameter=6.3mm, height=7mm, Electrolytic Capacitor")
 		(tags "CP Radial series Radial pin pitch 2.50mm diameter 6.3mm height 7mm Electrolytic Capacitor")
@@
 	)
 	(segment
-		(start 108.03 55.706)
-		(end 105.156 52.832)
+		(start 117.856 55.706)
+		(end 108.538 55.706)
 		(width 2.5)
 		(layer "B.Cu")
@@
 	)
 	(segment
-		(start 117.856 55.706)
-		(end 108.03 55.706)
+		(start 108.966 57.658)
+		(end 108.966 56.134)
+		(width 2.5)
+		(layer "B.Cu")
+		(net 1)
+	)
+	(segment
+		(start 108.966 56.134)
+		(end 108.538 55.706)
+		(width 2.5)
+		(layer "B.Cu")
+		(net 1)
+	)
+	(segment
+		(start 108.538 55.706)
+		(end 105.664 52.832)
 		(width 2.5)
 		(layer "B.Cu")
@@
 	)
 	(segment
-		(start 92.456 54.61)
-		(end 93.218 55.372)
-		(width 0.75)
-		(layer "B.Cu")
-		(net 2)
-	)
-	(segment
 		(start 58.928 62.992)
 		(end 64.389 68.453)
@@
 	)
 	(segment
-		(start 98.338 46.843)
-		(end 98.338 45.954)
+		(start 98.806 46.843)
+		(end 98.806 45.954)
 		(width 2)
 		(layer "B.Cu")
@@
 	)
 	(segment
-		(start 81.7372 46.9138)
-		(end 81.0514 47.5996)
-		(width 0.35)
-		(layer "B.Cu")
-		(net 2)
-	)
-	(segment
-		(start 98.338 44.557)
-		(end 98.338 46.843)
+		(start 98.806 44.557)
+		(end 98.806 46.843)
 		(width 0.5)
 		(layer "B.Cu")
@@
 	)
 	(segment
-		(start 66.1924 47.5996)
-		(end 66.167 47.625)
-		(width 0.35)
-		(layer "B.Cu")
-		(net 2)
-	)
-	(segment
 		(start 80.238 68.453)
 		(end 80.238 66.583)
@@
 	)
 	(segment
-		(start 93.218 55.372)
-		(end 101.6 55.372)
-		(width 0.75)
+		(start 81.0514 47.5996)
+		(end 66.1924 47.5996)
+		(width 0.35)
 		(layer "B.Cu")
 		(net 2)
@@
 	)
 	(segment
-		(start 98.338 44.557)
-		(end 97.723 43.942)
-		(width 0.35)
+		(start 80.238 66.583)
+		(end 80.212 66.557)
+		(width 0.5)
 		(layer "B.Cu")
 		(net 2)
 	)
 	(segment
-		(start 80.238 66.583)
-		(end 80.212 66.557)
-		(width 0.5)
+		(start 81.7372 46.9138)
+		(end 81.0514 47.5996)
+		(width 0.35)
 		(layer "B.Cu")
 		(net 2)
@@
 	)
 	(segment
+		(start 98.806 44.557)
+		(end 98.191 43.942)
+		(width 0.35)
+		(layer "B.Cu")
+		(net 2)
+	)
+	(segment
 		(start 80.238 70.375)
 		(end 80.238 68.453)
@@
 	)
 	(segment
+		(start 91.3892 48.9712)
+		(end 92.456 50.038)
+		(width 0.75)
+		(layer "B.Cu")
+		(net 2)
+	)
+	(segment
+		(start 83.82 48.9712)
+		(end 91.3892 48.9712)
+		(width 0.75)
+		(layer "B.Cu")
+		(net 2)
+	)
+	(segment
 		(start 86.36 65.278)
 		(end 85.081 66.557)
@@
 	)
 	(segment
-		(start 97.723 43.942)
-		(end 82.9056 43.942)
-		(width 0.35)
-		(layer "B.Cu")
-		(net 2)
-	)
-	(segment
 		(start 78.323 51.108)
 		(end 78.323 49.784)
@@
 	)
 	(segment
-		(start 81.7372 45.1104)
-		(end 81.7372 46.9138)
-		(width 0.35)
-		(layer "B.Cu")
-		(net 2)
-	)
-	(segment
 		(start 83.338 70.375)
 		(end 83.346 70.367)
@@
 	)
 	(segment
-		(start 83.82 48.9712)
-		(end 91.3892 48.9712)
-		(width 0.75)
-		(layer "B.Cu")
-		(net 2)
-	)
-	(segment
 		(start 79.9338 49.784)
 		(end 78.323 49.784)
@@
 	)
 	(segment
+		(start 81.7372 45.1104)
+		(end 81.7372 46.9138)
+		(width 0.35)
+		(layer "B.Cu")
+		(net 2)
+	)
+	(segment
+		(start 82.9056 43.942)
+		(end 81.7372 45.1104)
+		(width 0.35)
+		(layer "B.Cu")
+		(net 2)
+	)
+	(segment
 		(start 116.84 78.232)
 		(end 113.792 78.232)
@@
 	)
 	(segment
+		(start 93.472 55.626)
+		(end 101.346 55.626)
+		(width 0.75)
+		(layer "B.Cu")
+		(net 2)
+	)
+	(segment
 		(start 120.904 79.248)
 		(end 120.904 92.71)
@@
 	)
 	(segment
-		(start 82.9056 43.942)
-		(end 81.7372 45.1104)
+		(start 66.1924 47.5996)
+		(end 66.167 47.625)
+		(width 0.35)
+		(layer "B.Cu")
+		(net 2)
+	)
+	(segment
+		(start 98.191 43.942)
+		(end 82.9056 43.942)
 		(width 0.35)
 		(layer "B.Cu")
@@
 	)
 	(segment
-		(start 81.0514 47.5996)
-		(end 66.1924 47.5996)
-		(width 0.35)
-		(layer "B.Cu")
-		(net 2)
-	)
-	(segment
-		(start 91.3892 48.9712)
-		(end 92.456 50.038)
-		(width 0.75)
-		(layer "B.Cu")
-		(net 2)
-	)
-	(segment
 		(start 83.82 48.9712)
 		(end 80.7466 48.9712)
@@
 	)
 	(segment
-		(start 92.456 50.038)
-		(end 92.456 54.61)
-		(width 0.75)
-		(layer "B.Cu")
-		(net 2)
-	)
-	(segment
 		(start 84.38 66.557)
 		(end 84.389 66.548)
@@
 	)
 	(segment
+		(start 92.456 54.61)
+		(end 93.472 55.626)
+		(width 0.75)
+		(layer "B.Cu")
+		(net 2)
+	)
+	(segment
+		(start 92.456 50.038)
+		(end 92.456 54.61)
+		(width 0.75)
+		(layer "B.Cu")
+		(net 2)
+	)
+	(segment
 		(start 117.856 66.548)
 		(end 118.618 67.31)
@@
 	)
 	(segment
-		(start 98.2595 52.832)
-		(end 94.996 52.832)
-		(width 1)
+		(start 93.218 45.974)
+		(end 93.472 46.228)
+		(width 2.5)
 		(layer "B.Cu")
 		(net 4)
 	)
 	(segment
-		(start 93.2688 46.0248)
+		(start 93.472 46.228)
 		(end 94.996 47.752)
-		(width 2.5)
+		(width 3)
 		(layer "B.Cu")
 		(net 4)
@@
 	(segment
 		(start 94.996 47.752)
-		(end 94.996 52.832)
+		(end 95.504 48.26)
 		(width 2.5)
 		(layer "B.Cu")
@@
 	)
 	(segment
-		(start 83.5722 46.0248)
-		(end 93.2688 46.0248)
+		(start 84.7852 45.974)
+		(end 93.218 45.974)
 		(width 2.5)
 		(layer "B.Cu")
 		(net 4)
 	)
+	(segment
+		(start 95.504 48.26)
+		(end 95.504 52.832)
+		(width 3)
+		(layer "B.Cu")
+		(net 4)
+	)
+	(segment
+		(start 84.7514 45.9402)
+		(end 84.7852 45.974)
+		(width 2)
+		(layer "B.Cu")
+		(net 4)
+	)
+	(segment
+		(start 83.423 45.9402)
+		(end 84.7514 45.9402)
+		(width 2)
+		(layer "B.Cu")
+		(net 4)
+	)
+	(segment
+		(start 98.2595 52.832)
+		(end 95.504 52.832)
+		(width 1)
+		(layer "B.Cu")
+		(net 4)
+	)
 	(via
 		(at 104.14 73.66)
@@
 	)
 	(segment
-		(start 100.838 46.843)
-		(end 100.838 44.089)
+		(start 101.306 46.843)
+		(end 101.306 44.089)
 		(width 2)
 		(layer "B.Cu")
@@
 	)
 	(segment
+		(start 81.4832 43.688)
+		(end 82.2452 42.926)
+		(width 0.75)
+		(layer "B.Cu")
+		(net 10)
+	)
+	(segment
 		(start 80.01 43.688)
 		(end 81.4832 43.688)
@@
 	)
 	(segment
-		(start 99.675 42.926)
-		(end 99.782 43.033)
+		(start 82.2452 42.926)
+		(end 100.143 42.926)
 		(width 0.75)
 		(layer "B.Cu")
@@
 	)
 	(segment
-		(start 81.4832 43.688)
-		(end 82.2452 42.926)
-		(width 0.75)
-		(layer "B.Cu")
-		(net 10)
-	)
-	(segment
 		(start 80.023 45.9402)
 		(end 80.023 43.701)
@@
 	)
 	(segment
-		(start 99.782 43.033)
-		(end 100.798 44.049)
+		(start 100.143 42.926)
+		(end 100.25 43.033)
 		(width 0.75)
 		(layer "B.Cu")
@@
 	)
 	(segment
-		(start 82.2452 42.926)
-		(end 99.675 42.926)
+		(start 100.25 43.033)
+		(end 101.266 44.049)
 		(width 0.75)
 		(layer "B.Cu")
