File: 3886_3/3886_3.kicad_sch (KiCad schematic)
At the start: 60 parts, among them J101 2, J102 2, J103 3, Q101 BT139-600E, Q102 BC817, Q103 BC807, U101 LM3886TF

Commit message: Add files via upload
Parts:
- R119, R120: value 10 -> 1
Changed lines of the file:
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@@
 	(text "DNP if jumper\nwire used"
 		(exclude_from_sim no)
-		(at 251.46 154.94 0)
+		(at 252.984 151.384 0)
 		(effects
 			(font
@@
 		(dnp no)
 		(property "Reference" "R120"
-			(at 252.73 143.51 90)
+			(at 252.222 137.16 90)
 			(effects
 				(font
@@
 			)
 		)
-		(property "Value" "10"
-			(at 258.064 143.51 90)
+		(property "Value" "1"
+			(at 257.81 137.16 90)
 			(effects
 				(font
@@
 		(dnp no)
 		(property "Reference" "R119"
-			(at 252.73 137.16 90)
+			(at 252.222 130.556 90)
 			(effects
 				(font
@@
 			)
 		)
-		(property "Value" "10"
-			(at 258.064 137.16 90)
+		(property "Value" "1"
+			(at 257.556 130.556 90)
 			(effects
 				(font
@@
 		(dnp no)
 		(property "Reference" "R121"
-			(at 252.73 151.13 90)
+			(at 252.476 144.526 90)
 			(effects
 				(font
@@
 		)
 		(property "Value" "0"
-			(at 258.064 151.13 90)
+			(at 257.81 144.526 90)
 			(effects
 				(font

Commit message: Add files via upload
Parts:
- removed C120, C121: 100n, Capacitor_SMD:C_1206_3216Metric_Pad1.33x1.80mm_HandSolder, symbol Device:C_Small
Changed lines of the file:
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@@
 	)
 	(junction
-		(at 219.71 29.21)
-		(diameter 0)
-		(color 0 0 0 0)
-	)
-	(junction
 		(at 229.87 44.45)
 		(diameter 0)
@@
 	)
 	(junction
-		(at 219.71 52.07)
-		(diameter 0)
-		(color 0 0 0 0)
-	)
-	(junction
 		(at 199.39 44.45)
 		(diameter 0)
@@
 	)
 	(junction
-		(at 219.71 19.05)
-		(diameter 0)
-		(color 0 0 0 0)
-	)
-	(junction
 		(at 119.38 121.92)
 		(diameter 0)
@@
 	)
 	(junction
-		(at 219.71 44.45)
-		(diameter 0)
-		(color 0 0 0 0)
-	)
-	(junction
 		(at 62.23 120.65)
 		(diameter 0)
@@
 	(wire
 		(pts
-			(xy 219.71 44.45) (xy 229.87 44.45)
-		)
-		(stroke
-			(width 0)
-			(type default)
-		)
-	)
-	(wire
-		(pts
 			(xy 264.16 25.4) (xy 266.7 25.4)
 		)
@@
 	(wire
 		(pts
-			(xy 209.55 52.07) (xy 219.71 52.07)
-		)
-		(stroke
-			(width 0)
-			(type default)
-		)
-	)
-	(wire
-		(pts
 			(xy 199.39 29.21) (xy 209.55 29.21)
 		)
@@
 	(wire
 		(pts
-			(xy 219.71 19.05) (xy 219.71 21.59)
-		)
-		(stroke
-			(width 0)
-			(type default)
-		)
-	)
-	(wire
-		(pts
 			(xy 104.14 99.06) (xy 104.14 102.87)
 		)
@@
 	(wire
 		(pts
-			(xy 219.71 19.05) (xy 229.87 19.05)
+			(xy 209.55 19.05) (xy 229.87 19.05)
 		)
 		(stroke
@@
 	(wire
 		(pts
-			(xy 209.55 44.45) (xy 219.71 44.45)
+			(xy 209.55 44.45) (xy 229.87 44.45)
 		)
 		(stroke
@@
 	(wire
 		(pts
-			(xy 219.71 50.8) (xy 219.71 52.07)
-		)
-		(stroke
-			(width 0)
-			(type default)
-		)
-	)
-	(wire
-		(pts
 			(xy 265.43 139.7) (xy 265.43 147.32)
 		)
@@
 	(wire
 		(pts
-			(xy 209.55 29.21) (xy 219.71 29.21)
-		)
-		(stroke
-			(width 0)
-			(type default)
-		)
-	)
-	(wire
-		(pts
 			(xy 191.77 33.02) (xy 191.77 34.29)
 		)
@@
 	(wire
 		(pts
-			(xy 219.71 44.45) (xy 219.71 45.72)
-		)
-		(stroke
-			(width 0)
-			(type default)
-		)
-	)
-	(wire
-		(pts
-			(xy 219.71 26.67) (xy 219.71 29.21)
-		)
-		(stroke
-			(width 0)
-			(type default)
-		)
-	)
-	(wire
-		(pts
 			(xy 191.77 52.07) (xy 191.77 53.34)
 		)
@@
 	(wire
 		(pts
-			(xy 209.55 19.05) (xy 219.71 19.05)
-		)
-		(stroke
-			(width 0)
-			(type default)
-		)
-	)
-	(wire
-		(pts
 			(xy 152.4 107.95) (xy 152.4 109.22)
 		)
@@
 	(wire
 		(pts
-			(xy 219.71 29.21) (xy 229.87 29.21)
+			(xy 209.55 29.21) (xy 229.87 29.21)
 		)
 		(stroke
@@
 	(wire
 		(pts
-			(xy 219.71 52.07) (xy 229.87 52.07)
+			(xy 209.55 52.07) (xy 229.87 52.07)
 		)
 		(stroke
@@
 	)
 	(symbol
-		(lib_id "Device:C_Small")
-		(at 219.71 48.26 180)
-		(unit 1)
-		(exclude_from_sim no)
-		(in_bom yes)
-		(on_board yes)
-		(dnp no)
-		(fields_autoplaced yes)
-		(property "Reference" "C121"
-			(at 222.25 46.9835 0)
-			(effects
-				(font
-					(size 1.27 1.27)
-				)
-				(justify right)
-			)
-		)
-		(property "Value" "100n"
-			(at 222.25 49.5235 0)
-			(effects
-				(font
-					(size 1.27 1.27)
-				)
-				(justify right)
-			)
-		)
-		(property "Footprint" "Capacitor_SMD:C_1206_3216Metric_Pad1.33x1.80mm_HandSolder"
-			(at 219.71 48.26 0)
-			(effects
-				(font
-					(size 1.27 1.27)
-				)
-				(hide yes)
-			)
-		)
-		(property "Datasheet" "~"
-			(at 219.71 48.26 0)
-			(effects
-				(font
-					(size 1.27 1.27)
-				)
-				(hide yes)
-			)
-		)
-		(property "Description" "X7R, 50V"
-			(at 219.71 48.26 0)
-			(effects
-				(font
-					(size 1.27 1.27)
-				)
-				(hide yes)
-			)
-		)
-		(pin "2"
-		)
-		(pin "1"
-		)
-		(instances
-			(project "3886_1"
-				(path "/e5e4cd80-f3a6-42ed-a9b8-872499a3dd49"
-					(reference "C121")
-					(unit 1)
-				)
-			)
-		)
-	)
-	(symbol
 		(lib_id "Device:R_Small")
 		(at 138.43 151.13 90)
@@
 					(unit 1)
 				)
-			)
-		)
-	)
-	(symbol
-		(lib_id "Device:C_Small")
-		(at 219.71 24.13 180)
-		(unit 1)
-		(exclude_from_sim no)
-		(in_bom yes)
-		(on_board yes)
-		(dnp no)
-		(fields_autoplaced yes)
-		(property "Reference" "C120"
-			(at 222.25 22.8535 0)
-			(effects
-				(font
-					(size 1.27 1.27)
-				)
-				(justify right)
-			)
-		)
-		(property "Value" "100n"
-			(at 222.25 25.3935 0)
-			(effects
-				(font
-					(size 1.27 1.27)
-				)
-				(justify right)
-			)
-		)
-		(property "Footprint" "Capacitor_SMD:C_1206_3216Metric_Pad1.33x1.80mm_HandSolder"
-			(at 219.71 24.13 0)
-			(effects
-				(font
-					(size 1.27 1.27)
-				)
-				(hide yes)
-			)
-		)
-		(property "Datasheet" "~"
-			(at 219.71 24.13 0)
-			(effects
-				(font
-					(size 1.27 1.27)
-				)
-				(hide yes)
-			)
-		)
-		(property "Description" "X7R, 50V"
-			(at 219.71 24.13 0)
-			(effects
-				(font
-					(size 1.27 1.27)
-				)
-				(hide yes)
-			)
-		)
-		(pin "2"
-		)
-		(pin "1"
-		)
-		(instances
-			(project "3886_1"
-				(path "/e5e4cd80-f3a6-42ed-a9b8-872499a3dd49"
-					(reference "C120")
-					(unit 1)
-				)

Commit message: Add files via upload
supply caps removed
Other:
- note added: "X7R!"
Changed lines of the file:
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@@
+		)
+	)
+	(text "X7R!"
+		(exclude_from_sim no)
+		(at 228.346 32.512 0)
+		(effects
+			(font
+				(size 1.27 1.27)
+			)
+			(justify left)
 		)
 	)

Commit message: Add files via upload
Other:
- note added: "Irms 1.5A fuse 3A, >20 A^2S"
- note removed: "Irms 1.5A fuse 3A, 20 A^2S"
Changed lines of the file:
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@@
 		)
 	)
-	(text "Irms 1.5A\nfuse 3A, 20 A^2S"
+	(text "Irms 1.5A\nfuse 3A, >20 A^2S"
 		(exclude_from_sim no)
 		(at 234.696 54.864 0)

Commit message: Add files via upload
Parts:
- removed R101: 0, Resistor_SMD:R_1206_3216Metric_Pad1.30x1.75mm_HandSolder, symbol Device:R_Small
Connections:
- net GND: now also J101.1 (Pin_1)
Changed lines of the file:
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@@
 	(wire
 		(pts
-			(xy 27.94 107.95) (xy 27.94 111.76)
+			(xy 27.94 99.06) (xy 27.94 111.76)
 		)
 		(stroke
@@
 	(wire
 		(pts
-			(xy 27.94 99.06) (xy 27.94 102.87)
-		)
-		(stroke
-			(width 0)
-			(type default)
-		)
-	)
-	(wire
-		(pts
 			(xy 133.35 187.96) (xy 134.62 187.96)
 		)
@@
 					(unit 1)
 				)
-			)
-		)
-	)
-	(symbol
-		(lib_id "Device:R_Small")
-		(at 27.94 105.41 0)
-		(unit 1)
-		(exclude_from_sim no)
-		(in_bom yes)
-		(on_board yes)
-		(dnp no)
-		(property "Reference" "R101"
-			(at 24.13 105.156 90)
-			(effects
-				(font
-					(size 1.27 1.27)
-				)
-			)
-		)
-		(property "Value" "0"
-			(at 25.908 105.156 90)
-			(effects
-				(font
-					(size 1.27 1.27)
-				)
-			)
-		)
-		(property "Footprint" "Resistor_SMD:R_1206_3216Metric_Pad1.30x1.75mm_HandSolder"
-			(at 27.94 105.41 0)
-			(effects
-				(font
-					(size 1.27 1.27)
-				)
-				(hide yes)
-			)
-		)
-		(property "Datasheet" "~"
-			(at 27.94 105.41 0)
-			(effects
-				(font
-					(size 1.27 1.27)
-				)
-				(hide yes)
-			)
-		)
-		(property "Description" "Resistor, small symbol"
-			(at 27.94 105.41 0)
-			(effects
-				(font
-					(size 1.27 1.27)
-				)
-				(hide yes)
-			)
-		)
-		(pin "1"
-		)
-		(pin "2"
-		)
-		(instances
-			(project "3886_3"
-				(path "/e5e4cd80-f3a6-42ed-a9b8-872499a3dd49"
-					(reference "R101")
-					(unit 1)
-				)
