File: PGA2311_3/PGA2311_3.kicad_pcb (KiCad board)
At the start: 2 copper layers, 234 x 58 mm, 205 parts, among them J201 3, J202 3, J203 2, J204 2, J301 Conn_01x16, J302 1, J303 Conn_01x02, J304 4, J305 4, J401 1, J402 3, J403 1, Q301 BC817-40, SW301 SW_Push, SW302 Encoder PEC11R, U201 OPA1678IDR, U202 CD74HCT4052B, U203 CD74HCT4052B, U204 LM337LM, U205 PGA2311UA, U206 LM317LIDR, U207 UA78L05AIDR, U301 TPS60403DBV, U302 WH1602B, U303 SN74LVC8T245DW, U304 STM32G070KBT6, U305 TLV1117-50IDC, U306 LP2985-33DBV, U307 SN74LVC2G17DBV

Commit message: Add files via upload
Routing:
- net Net-(C220-Pad2): track 19.2 -> 18.4 mm

Commit message: Add files via upload
Parts:
- moved C314 0.57 mm to (205.7, 63.8)
- moved C302 0.25 mm to (125.0, 42.2)
Routing:
- net Net-(C314-Pad1): track 15.0 -> 15.7 mm
- net GND: vias 258 -> 253
Changed lines of the file:
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@@
 		(pad "" thru_hole circle
 			(at -5.4991 0)
-			(size 5.5 5.5)
+			(size 6 6)
 			(drill 3)
 			(layers "*.Cu" "*.Mask")
@@
 		(pad "" thru_hole circle
 			(at -5.4991 31.0007)
-			(size 5.5 5.5)
+			(size 6 6)
 			(drill 3)
 			(layers "*.Cu" "*.Mask")
@@
 		(pad "" thru_hole circle
 			(at 69.49948 31.0007)
-			(size 5.5 5.5)
+			(size 6 6)
 			(drill 3)
 			(layers "*.Cu" "*.Mask")
@@
 		(pad "" thru_hole circle
 			(at 69.5 0)
-			(size 5.5 5.5)
+			(size 6 6)
 			(drill 3)
 			(layers "*.Cu" "*.Mask")
@@
 		(tags "resistor handsolder")
 		(property "Reference" "R322"
-			(at 0.508 -1.524 0)
+			(at 0.635 -1.524 0)
 			(layer "F.SilkS")
 			(effects
@@
 		(tags "CP Radial series Radial pin pitch 3.50mm diameter 8mm height 12mm Electrolytic Capacitor")
 		(property "Reference" "C412"
-			(at 6.858 4.191 0)
+			(at 6.223 4.318 0)
 			(layer "F.SilkS")
 			(effects
@@
 		(tags "CP Radial series Radial pin pitch 3.50mm diameter 8mm height 12mm Electrolytic Capacitor")
 		(property "Reference" "C411"
-			(at 6.35 4.191 0)
+			(at 5.842 4.318 0)
 			(layer "F.SilkS")
 			(effects
@@
 		(tags "CP Radial series Radial pin pitch 3.50mm diameter 8mm height 12mm Electrolytic Capacitor")
 		(property "Reference" "C408"
-			(at 4.826 4.699 0)
+			(at 4.699 4.699 0)
 			(layer "F.SilkS")
 			(effects
@@
 		(tags "resistor handsolder")
 		(property "Reference" "R340"
-			(at -3.81 -0.508 90)
+			(at -3.81 -0.635 90)
 			(layer "B.SilkS")
 			(effects
@@
 		(tags "capacitor handsolder")
 		(property "Reference" "C310"
-			(at 1.397 -1.905 90)
+			(at 0.762 -1.651 90)
 			(layer "B.SilkS")
 			(effects
@@
 	(footprint "Capacitor_SMD:C_0805_2012Metric_Pad1.18x1.45mm_HandSolder"
 		(layer "B.Cu")
-		(at 125.222 42.164 180)
+		(at 124.968 42.164 180)
 		(descr "Capacitor SMD 0805 (2012 Metric), square (rectangular) end terminal, IPC-7351 nominal with elongated pad for handsoldering. (Body size source: IPC-SM-782 page 76, https://www.pcb-3d.com/wordpress/wp-content/uploads/ipc-sm-782a_amendment_1_and_2.pdf, https://docs.google.com/spreadsheets/d/1BsfQQcO9C6DZCsRaXUlFlo91Tg2WpOkGARC1WS5S8t0/edit?usp=sharing), generated with kicad-footprint-generator")
 		(tags "capacitor handsolder")
@@
 		(tags "capacitor handsolder")
 		(property "Reference" "C318"
-			(at -1.397 -1.651 90)
+			(at 0 -2.667 90)
 			(layer "B.SilkS")
 			(effects
@@
 	(footprint "Capacitor_SMD:C_0805_2012Metric_Pad1.18x1.45mm_HandSolder"
 		(layer "B.Cu")
-		(at 205.486 64.262 -90)
+		(at 205.74 63.754 -90)
 		(descr "Capacitor SMD 0805 (2012 Metric), square (rectangular) end terminal, IPC-7351 nominal with elongated pad for handsoldering. (Body size source: IPC-SM-782 page 76, https://www.pcb-3d.com/wordpress/wp-content/uploads/ipc-sm-782a_amendment_1_and_2.pdf, https://docs.google.com/spreadsheets/d/1BsfQQcO9C6DZCsRaXUlFlo91Tg2WpOkGARC1WS5S8t0/edit?usp=sharing), generated with kicad-footprint-generator")
 		(tags "capacitor handsolder")
@@
 		(tags "capacitor handsolder")
 		(property "Reference" "C317"
-			(at -0.889 -1.524 90)
+			(at 0.127 1.778 90)
 			(layer "B.SilkS")
 			(effects
@@
 	)
 	(gr_text "GND"
-		(at 132.842 37.973 90)
+		(at 134.874 35.306 90)
 		(layer "B.SilkS")
 		(effects
@@
 	)
 	(via
-		(at 206.248 24.384)
-		(size 1)
-		(drill 0.5)
-		(layers "F.Cu" "B.Cu")
-		(free yes)
-		(net 1)
-	)
-	(via
 		(at 48.133 43.434)
 		(size 1)
@@
 	)
 	(via
-		(at 125.349 38.735)
+		(at 125.222 38.735)
 		(size 1)
 		(drill 0.5)
@@
 	)
 	(via
-		(at 207.518 36.576)
+		(at 207.899 36.576)
 		(size 1)
 		(drill 0.5)
@@
 	)
 	(via
-		(at 207.518 42.291)
+		(at 207.899 42.291)
 		(size 1)
 		(drill 0.5)
@@
 	)
 	(via
-		(at 200.533 24.384)
-		(size 1)
-		(drill 0.5)
-		(layers "F.Cu" "B.Cu")
-		(free yes)
-		(net 1)
-	)
-	(via
 		(at 35.5385 36.449)
 		(size 1)
@@
 	)
 	(via
-		(at 204.089 31.496)
-		(size 1)
-		(drill 0.5)
-		(layers "F.Cu" "B.Cu")
-		(free yes)
-		(net 1)
-	)
-	(via
 		(at 49.911 31.75)
 		(size 1)
@@
 	)
 	(via
-		(at 205.613 31.496)
-		(size 1)
-		(drill 0.5)
-		(layers "F.Cu" "B.Cu")
-		(free yes)
-		(net 1)
-	)
-	(via
 		(at 106.299 22.352)
 		(size 1)
@@
 	)
 	(via
-		(at 202.057 34.925)
+		(at 202.184 34.798)
 		(size 1)
 		(drill 0.5)
@@
 	)
 	(via
-		(at 204.089 34.925)
-		(size 1)
-		(drill 0.5)
-		(layers "F.Cu" "B.Cu")
-		(free yes)
-		(net 1)
-	)
-	(via
 		(at 91.948 74.422)
 		(size 1)
@@
 		(drill 0.5)
 		(layers "F.Cu" "B.Cu")
+		(tenting none)
 		(net 119)
 	)
@@
 	)
 	(segment
-		(start 206.8615 63.2245)
-		(end 205.486 63.2245)
-		(width 0.5)
+		(start 206.375 62.738)
+		(end 207.01 62.738)
+		(width 0.35)
 		(layer "B.Cu")
 		(net 133)
 	)
 	(segment
-		(start 210.82 69.596)
-		(end 207.264 66.04)
-		(width 0.35)
+		(start 201.549 61.96)
+		(end 202.749657 61.96)
+		(width 0.5)
 		(layer "B.Cu")
 		(net 133)
 	)
 	(segment
-		(start 204.014157 63.2245)
-		(end 205.486 63.2245)
+		(start 203.506157 62.7165)
+		(end 205.74 62.7165)
 		(width 0.5)
 		(layer "B.Cu")
@@
 	)
 	(segment
-		(start 207.264 63.627)
-		(end 206.8615 63.2245)
+		(start 207.264 66.04)
+		(end 210.82 69.596)
 		(width 0.35)
 		(layer "B.Cu")
@@
 	)
 	(segment
-		(start 207.264 66.04)
-		(end 207.264 63.627)
+		(start 207.264 62.992)
+		(end 207.264 66.04)
 		(width 0.35)
 		(layer "B.Cu")
@@
 	(segment
 		(start 202.749657 61.96)
-		(end 204.014157 63.2245)
+		(end 203.506157 62.7165)
 		(width 0.5)
 		(layer "B.Cu")
@@
 	)
 	(segment
-		(start 201.549 61.96)
-		(end 202.749657 61.96)
+		(start 206.7345 62.7165)
+		(end 205.74 62.7165)
 		(width 0.5)
 		(layer "B.Cu")
 		(net 133)
+	)
+	(segment
+		(start 207.01 62.738)
+		(end 207.264 62.992)
+		(width 0.35)
+		(layer "B.Cu")
+		(net 133)

Commit message: Add files via upload
Parts:
- U202, U203: value CD74HCT4052B -> CD74HCT4052
- moved R327 0.74 mm to (237.9, 50.7)
- moved R229 0.64 mm to (30.4, 39.9)
- moved R343 0.63 mm to (235.5, 63.6)
- moved R302 0.51 mm to (133.9, 42.9)
- moved C228 0.25 mm to (30.5, 35.3)
- moved C303 0.25 mm to (137.9, 43.4)
- moved C302 0.13 mm to (124.8, 42.2)
Routing:
- net /analog/+5VA: track 128.5 -> 127.8 mm
- net Net-(D301-A): track 4.08 -> 4.72 mm
- net GND: track 149.3 -> 148.7 mm
- net Net-(R302-Pad2): track 13.2 -> 12.7 mm

Commit message: Add files via upload
lm337 load resistor moved, pga2311 output resistor moved
Parts:
- R224: moved to B.Cu
- moved R224 16.6 mm to (79.0, 57.5)
- moved R227 5.71 mm to (43.9, 53.8), turned to -45 degrees
- moved R228 5.34 mm to (44.1, 37.5), turned to 45 degrees
- moved C236 0.89 mm to (51.4, 26.4)
- moved R206 0.76 mm to (77.3, 23.5)
- moved R233 0.13 mm to (47.5, 31.6)
Routing:
- net Net-(U205-V_{OUT}L): track 20.0 -> 8.13 mm, vias 1 -> 0
- net Net-(U205-V_{OUT}R): track 15.5 -> 8.39 mm, vias 1 -> 0
- net Net-(J204-Pin_1): track 21.2 -> 26.9 mm, vias 0 -> 1
- net Net-(J203-Pin_1): track 19.2 -> 24.7 mm, vias 0 -> 1
- net GND: track 148.7 -> 145.4 mm, vias 253 -> 250
- net /analog/+5VA: track 127.8 -> 129.7 mm
- net Net-(U203-VDD): track 7.78 -> 7.02 mm

Commit message: Add files via upload
Routing:
- net GND: track 145.4 -> 142.4 mm, vias 250 -> 249
