File: PGA2311_3/analog.kicad_sch (KiCad schematic)
At the start: 91 parts, among them J201 3, J202 3, J203 2, J204 2, J205 2, J206 2, J207 2, J208 2, U201 OPA1678IDR, U202 CD74HCT4052, U203 CD74HCT4052, U204 LM337LM, U205 PGA2311UA, U206 LM317LIDR, U207 UA78L05AIDR

Commit message: Add files via upload
Parts:
- removed H201: MountingHole_Pad, MountingHole:MountingHole_2.5mm_Pad_Via, symbol Mechanical:MountingHole_Pad
Changed lines of the file:
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@@
 	(wire
 		(pts
-			(xy 257.81 64.77) (xy 257.81 67.31)
-		)
-		(stroke
-			(width 0)
-			(type default)
-		)
-	)
-	(wire
-		(pts
 			(xy 95.25 74.93) (xy 97.79 74.93)
 		)
@@
 	)
 	(symbol
-		(lib_id "Mechanical:MountingHole_Pad")
-		(at 257.81 62.23 0)
-		(unit 1)
-		(exclude_from_sim no)
-		(in_bom no)
-		(on_board yes)
-		(dnp no)
-		(fields_autoplaced yes)
-		(property "Reference" "H201"
-			(at 260.35 59.6899 0)
-			(effects
-				(font
-					(size 1.27 1.27)
-				)
-				(justify left)
-			)
-		)
-		(property "Value" "MountingHole_Pad"
-			(at 260.35 62.2299 0)
-			(effects
-				(font
-					(size 1.27 1.27)
-				)
-				(justify left)
-			)
-		)
-		(property "Footprint" "MountingHole:MountingHole_2.5mm_Pad_Via"
-			(at 257.81 62.23 0)
-			(effects
-				(font
-					(size 1.27 1.27)
-				)
-				(hide yes)
-			)
-		)
-		(property "Datasheet" "~"
-			(at 257.81 62.23 0)
-			(effects
-				(font
-					(size 1.27 1.27)
-				)
-				(hide yes)
-			)
-		)
-		(property "Description" "Mounting Hole with connection"
-			(at 257.81 62.23 0)
-			(effects
-				(font
-					(size 1.27 1.27)
-				)
-				(hide yes)
-			)
-		)
-		(pin "1"
-		)
-		(instances
-			(project ""
-				(path "/e4f5d1ca-8b46-4ca2-bb25-7f237c56d603/417e42a4-c07c-47f8-ba75-79030ad924cb"
-					(reference "H201")
-					(unit 1)
-				)
-			)
-		)
-	)
-	(symbol
 		(lib_id "power:GND")
 		(at 237.49 41.91 0)
@@
 					(unit 1)
 				)
-			)
-		)
-	)
-	(symbol
-		(lib_id "power:GND")
-		(at 257.81 67.31 0)
-		(unit 1)
-		(exclude_from_sim no)
-		(in_bom yes)
-		(on_board yes)
-		(dnp no)
-		(property "Reference" "#PWR0203"
-			(at 257.81 73.66 0)
-			(effects
-				(font
-					(size 1.27 1.27)
-				)
-				(hide yes)
-			)
-		)
-		(property "Value" "GND"
-			(at 262.128 69.342 0)
-			(effects
-				(font
-					(size 1.27 1.27)
-				)
-			)
-		)
-		(property "Footprint" ""
-			(at 257.81 67.31 0)
-			(effects
-				(font
-					(size 1.27 1.27)
-				)
-				(hide yes)
-			)
-		)
-		(property "Datasheet" ""
-			(at 257.81 67.31 0)
-			(effects
-				(font
-					(size 1.27 1.27)
-				)
-				(hide yes)
-			)
-		)
-		(property "Description" "Power symbol creates a global label with name \"GND\" , ground"
-			(at 257.81 67.31 0)
-			(effects
-				(font
-					(size 1.27 1.27)
-				)
-				(hide yes)
-			)
-		)
-		(pin "1"
-		)
-		(instances
-			(project "PGA2311_3"
-				(path "/e4f5d1ca-8b46-4ca2-bb25-7f237c56d603/417e42a4-c07c-47f8-ba75-79030ad924cb"
-					(reference "#PWR0203")
-					(unit 1)
-				)

Commit message: Add files via upload
Parts:
- R220, R221: value 100 -> 220
Other:
- note added: "-3dB 10Hz - 350 kHz"
- note removed: "-3dB 10Hz - 400 kHz"
Changed lines of the file:
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@@
 		)
 	)
-	(text " -3dB 10Hz - 400 kHz"
+	(text " -3dB 10Hz - 350 kHz"
 		(exclude_from_sim no)
 		(at 145.288 48.006 0)
@@
 			)
 		)
-		(property "Value" "100"
+		(property "Value" "220"
 			(at 129.54 54.61 90)
 			(effects
@@
 			)
 		)
-		(property "Value" "100"
+		(property "Value" "220"
 			(at 130.81 80.01 90)
 			(effects

Commit message: Add files via upload
v2.6 +-5V output capacitor increased and reverse diodes added
Parts:
- added D101, D202: 1N5819, Diode_SMD:D_SOD-123, symbol Diode:1N5819
- C224, C236: value 22u -> 33u
Connections:
- net +5VA: now also D101.2 (A)
- net -5VA: now also D202.1 (K)
- net at C228.1, C231.1, R226.2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: now also D101.1 (K)
- net at C210.1, C213.1, R207.2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: now also D202.2 (A)
Other:
- note added: "9 mA"
- note removed: "4 mA"
Changed lines of the file:
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@@
 		(title "Preamp2311")
 		(date "08.2026")
-		(rev "2_5")
+		(rev "2_6")
 		(company "DMSDL")
 		(comment 1 "designed by Oleg Voitovich")
 		(comment 2 "CERN-OHL-S v2 license")
 	)
-	(text "4 mA"
+	(text "9 mA"
 		(exclude_from_sim no)
-		(at 203.708 136.652 0)
+		(at 201.168 136.906 0)
 		(effects
 			(font
@@
 		)
 	)
-	(text "4 mA"
+	(text "9 mA"
 		(exclude_from_sim no)
-		(at 96.52 169.164 0)
+		(at 91.44 169.164 0)
 		(effects
 			(font
@@
 	)
 	(junction
+		(at 207.01 142.24)
+		(diameter 0)
+		(color 0 0 0 0)
+	)
+	(junction
 		(at 210.82 54.61)
 		(diameter 0)
@@
 	(wire
 		(pts
+			(xy 207.01 132.08) (xy 207.01 142.24)
+		)
+		(stroke
+			(width 0)
+			(type default)
+		)
+	)
+	(wire
+		(pts
 			(xy 107.95 27.94) (xy 107.95 29.21)
 		)
@@
 	(wire
 		(pts
+			(xy 226.06 132.08) (xy 226.06 142.24)
+		)
+		(stroke
+			(width 0)
+			(type default)
+		)
+	)
+	(wire
+		(pts
 			(xy 101.6 50.8) (xy 106.68 50.8)
 		)
@@
 	(wire
 		(pts
+			(xy 95.25 161.29) (xy 95.25 172.72)
+		)
+		(stroke
+			(width 0)
+			(type default)
+		)
+	)
+	(wire
+		(pts
 			(xy 41.91 163.83) (xy 41.91 166.37)
 		)
@@
 	(wire
 		(pts
+			(xy 111.76 161.29) (xy 118.11 161.29)
+		)
+		(stroke
+			(width 0)
+			(type default)
+		)
+	)
+	(wire
+		(pts
 			(xy 176.53 97.79) (xy 176.53 99.06)
 		)
@@
 	(wire
 		(pts
+			(xy 118.11 161.29) (xy 118.11 172.72)
+		)
+		(stroke
+			(width 0)
+			(type default)
+		)
+	)
+	(wire
+		(pts
 			(xy 105.41 81.28) (xy 111.76 81.28)
 		)
@@
 	(wire
 		(pts
+			(xy 104.14 161.29) (xy 95.25 161.29)
+		)
+		(stroke
+			(width 0)
+			(type default)
+		)
+	)
+	(wire
+		(pts
 			(xy 198.12 87.63) (xy 209.55 87.63)
 		)
@@
 	(wire
 		(pts
+			(xy 210.82 132.08) (xy 207.01 132.08)
+		)
+		(stroke
+			(width 0)
+			(type default)
+		)
+	)
+	(wire
+		(pts
 			(xy 96.52 43.18) (xy 97.79 43.18)
 		)
@@
 	(wire
 		(pts
+			(xy 207.01 142.24) (xy 208.28 142.24)
+		)
+		(stroke
+			(width 0)
+			(type default)
+		)
+	)
+	(wire
+		(pts
 			(xy 124.46 81.28) (xy 124.46 91.44)
 		)
@@
 	(wire
 		(pts
-			(xy 203.2 142.24) (xy 208.28 142.24)
+			(xy 203.2 142.24) (xy 207.01 142.24)
 		)
 		(stroke
@@
 	(wire
 		(pts
+			(xy 218.44 132.08) (xy 226.06 132.08)
+		)
+		(stroke
+			(width 0)
+			(type default)
+		)
+	)
+	(wire
+		(pts
 			(xy 97.79 133.35) (xy 97.79 134.62)
 		)
@@
 	)
 	(symbol
+		(lib_id "Diode:1N5819")
+		(at 107.95 161.29 180)
+		(unit 1)
+		(exclude_from_sim no)
+		(in_bom yes)
+		(on_board yes)
+		(dnp no)
+		(fields_autoplaced yes)
+		(property "Reference" "D202"
+			(at 108.2675 154.94 0)
+			(effects
+				(font
+					(size 1.27 1.27)
+				)
+			)
+		)
+		(property "Value" "1N5819"
+			(at 108.2675 157.48 0)
+			(effects
+				(font
+					(size 1.27 1.27)
+				)
+			)
+		)
+		(property "Footprint" "Diode_SMD:D_SOD-123"
+			(at 107.95 156.845 0)
+			(effects
+				(font
+					(size 1.27 1.27)
+				)
+				(hide yes)
+			)
+		)
+		(property "Datasheet" "http://www.vishay.com/docs/88525/1n5817.pdf"
+			(at 107.95 161.29 0)
+			(effects
+				(font
+					(size 1.27 1.27)
+				)
+				(hide yes)
+			)
+		)
+		(property "Description" "40V 1A Schottky Barrier Rectifier Diode, DO-41"
+			(at 107.95 161.29 0)
+			(effects
+				(font
+					(size 1.27 1.27)
+				)
+				(hide yes)
+			)
+		)
+		(pin "1"
+		)
+		(pin "2"
+		)
+		(instances
+			(project "PGA2311_3"
+				(path "/e4f5d1ca-8b46-4ca2-bb25-7f237c56d603/417e42a4-c07c-47f8-ba75-79030ad924cb"
+					(reference "D202")
+					(unit 1)
+				)
+			)
+		)
+	)
+	(symbol
 		(lib_id "Device:C_Small")
 		(at 36.83 66.04 90)
@@
 	)
 	(symbol
+		(lib_id "Diode:1N5819")
+		(at 214.63 132.08 0)
+		(unit 1)
+		(exclude_from_sim no)
+		(in_bom yes)
+		(on_board yes)
+		(dnp no)
+		(fields_autoplaced yes)
+		(property "Reference" "D101"
+			(at 214.3125 125.73 0)
+			(effects
+				(font
+					(size 1.27 1.27)
+				)
+			)
+		)
+		(property "Value" "1N5819"
+			(at 214.3125 128.27 0)
+			(effects
+				(font
+					(size 1.27 1.27)
+				)
+			)
+		)
+		(property "Footprint" "Diode_SMD:D_SOD-123"
+			(at 214.63 136.525 0)
+			(effects
+				(font
+					(size 1.27 1.27)
+				)
+				(hide yes)
+			)
+		)
+		(property "Datasheet" "http://www.vishay.com/docs/88525/1n5817.pdf"
+			(at 214.63 132.08 0)
+			(effects
+				(font
+					(size 1.27 1.27)
+				)
+				(hide yes)
+			)
+		)
+		(property "Description" "40V 1A Schottky Barrier Rectifier Diode, DO-41"
+			(at 214.63 132.08 0)
+			(effects
+				(font
+					(size 1.27 1.27)
+				)
+				(hide yes)
+			)
+		)
+		(pin "1"
+		)
+		(pin "2"
+		)
+		(instances
+			(project "PGA2311_3"
+				(path "/e4f5d1ca-8b46-4ca2-bb25-7f237c56d603/417e42a4-c07c-47f8-ba75-79030ad924cb"
+					(reference "D101")
+					(unit 1)
+				)
+			)
+		)
+	)
+	(symbol
 		(lib_id "power:GND")
 		(at 41.91 172.72 0)
@@
 			)
 		)
-		(property "Value" "22u"
+		(property "Value" "33u"
 			(at 140.97 165.646 0)
 			(effects
@@
 			)
 		)
-		(property "Value" "22u"
+		(property "Value" "33u"
 			(at 251.46 132.8038 0)
 			(effects

Commit message: Add files via upload
Parts:
- added H201, H202, H203, H204: MountingHole, MountingHole:MountingHole_2.7mm_M2.5, symbol Mechanical:MountingHole

Commit message: Add files via upload
Parts:
- removed C233: 10u, Capacitor_SMD:C_0805_2012Metric_Pad1.18x1.45mm_HandSolder, symbol Device:C_Small
- C234: value 0 -> 10u
Changed lines of the file:
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@@
 	)
 	(junction
-		(at 228.6 29.21)
-		(diameter 0)
-		(color 0 0 0 0)
-	)
-	(junction
 		(at 226.06 142.24)
 		(diameter 0)
@@
 	(wire
 		(pts
-			(xy 228.6 38.1) (xy 228.6 41.91)
-		)
-		(stroke
-			(width 0)
-			(type default)
-		)
-	)
-	(wire
-		(pts
 			(xy 128.27 110.49) (xy 128.27 113.03)
 		)
@@
 	(wire
 		(pts
-			(xy 228.6 29.21) (xy 237.49 29.21)
-		)
-		(stroke
-			(width 0)
-			(type default)
-		)
-	)
-	(wire
-		(pts
 			(xy 132.08 175.26) (xy 132.08 172.72)
 		)
@@
 	(wire
 		(pts
-			(xy 226.06 29.21) (xy 228.6 29.21)
+			(xy 226.06 29.21) (xy 237.49 29.21)
 		)
 		(stroke
@@
 	(wire
 		(pts
-			(xy 228.6 29.21) (xy 228.6 33.02)
-		)
-		(stroke
-			(width 0)
-			(type default)
-		)
-	)
-	(wire
-		(pts
 			(xy 203.2 142.24) (xy 203.2 144.78)
 		)
@@
 			)
 		)
-		(property "Value" "0"
+		(property "Value" "10u"
 			(at 240.03 36.8362 0)
 			(effects
@@
 	)
 	(symbol
-		(lib_id "Device:C_Small")
-		(at 228.6 35.56 0)
-		(unit 1)
-		(exclude_from_sim no)
-		(in_bom yes)
-		(on_board yes)
-		(dnp no)
-		(fields_autoplaced yes)
-		(property "Reference" "C233"
-			(at 231.14 34.2962 0)
-			(effects
-				(font
-					(size 1.27 1.27)
-				)
-				(justify left)
-			)
-		)
-		(property "Value" "10u"
-			(at 231.14 36.8362 0)
-			(effects
-				(font
-					(size 1.27 1.27)
-				)
-				(justify left)
-			)
-		)
-		(property "Footprint" "Capacitor_SMD:C_0805_2012Metric_Pad1.18x1.45mm_HandSolder"
-			(at 228.6 35.56 0)
-			(effects
-				(font
-					(size 1.27 1.27)
-				)
-				(hide yes)
-			)
-		)
-		(property "Datasheet" "~"
-			(at 228.6 35.56 0)
-			(effects
-				(font
-					(size 1.27 1.27)
-				)
-				(hide yes)
-			)
-		)
-		(property "Description" "Unpolarized capacitor, small symbol"
-			(at 228.6 35.56 0)
-			(effects
-				(font
-					(size 1.27 1.27)
-				)
-				(hide yes)
-			)
-		)
-		(pin "1"
-		)
-		(pin "2"
-		)
-		(instances
-			(project "PGA2311_3"
-				(path "/e4f5d1ca-8b46-4ca2-bb25-7f237c56d603/417e42a4-c07c-47f8-ba75-79030ad924cb"
-					(reference "C233")
-					(unit 1)
-				)
-			)
-		)
-	)
-	(symbol
 		(lib_id "Device:R_Small")
 		(at 114.3 72.39 90)
@@
 					(unit 1)
 				)
-			)
-		)
-	)
-	(symbol
-		(lib_id "power:GND")
-		(at 228.6 41.91 0)
-		(unit 1)
-		(exclude_from_sim no)
-		(in_bom yes)
-		(on_board yes)
-		(dnp no)
-		(property "Reference" "#PWR0253"
-			(at 228.6 48.26 0)
-			(effects
-				(font
-					(size 1.27 1.27)
-				)
-				(hide yes)
-			)
-		)
-		(property "Value" "GND"
-			(at 232.918 43.942 0)
-			(effects
-				(font
-					(size 1.27 1.27)
-				)
-			)
-		)
-		(property "Footprint" ""
-			(at 228.6 41.91 0)
-			(effects
-				(font
-					(size 1.27 1.27)
-				)
-				(hide yes)
-			)
-		)
-		(property "Datasheet" ""
-			(at 228.6 41.91 0)
-			(effects
-				(font
-					(size 1.27 1.27)
-				)
-				(hide yes)
-			)
-		)
-		(property "Description" "Power symbol creates a global label with name \"GND\" , ground"
-			(at 228.6 41.91 0)
-			(effects
-				(font
-					(size 1.27 1.27)
-				)
-				(hide yes)
-			)
-		)
-		(pin "1"
-		)
-		(instances
-			(project "PGA2311_3"
-				(path "/e4f5d1ca-8b46-4ca2-bb25-7f237c56d603/417e42a4-c07c-47f8-ba75-79030ad924cb"
-					(reference "#PWR0253")
-					(unit 1)
-				)
